File: hardware/iot-open-soil-moisture-sensor-lora-samd10.kicad_sch (KiCad schematic)
At the start: 40 parts, among them J1 ARM-JTAG-SWD-10, J2 Conn_01x04_Pin, J3 Conn_01x04_Pin, Q1 IRLML6401, Q2 NTJD1155LT1, U1 ATSAMD10D14A-SS, U2 TPD2E009DBZR, U3 TPD2E009DBZR, U4 Ai-Thinker-Ra-02, Y1 KX-327NHT

Commit message: add PCB signs
Connections:
- net SCL1: now also R4.2, U2.1 (D+); no longer R5.2, U2.2 (D-)
- net SCL2: now also R6.2, U3.1 (D+); no longer R7.2, U3.2 (D-)
- net SDA1: now also R5.2, U2.2 (D-); no longer R4.2, U2.1 (D+)
- net SDA2: now also R7.2, U3.2 (D-); no longer R6.2, U3.1 (D+)
Changed lines of the file:
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@@
     (effects (font (size 2 2) (thickness 0.254) bold) (justify left bottom))
   )
-  (global_label "SCL2" (shape input) (at 222.25 34.29 0) (fields_autoplaced)
-    (effects (font (size 1.27 1.27)) (justify left))
-    (property "Intersheetrefs" "${INTERSHEET_REFS}" (at 229.8729 34.29 0)
-      (effects (font (size 1.27 1.27)) (justify left) hide)
+  (global_label "SCL2" (shape input) (at 196.85 34.29 180) (fields_autoplaced)
+    (effects (font (size 1.27 1.27)) (justify right))
+    (property "Intersheetrefs" "${INTERSHEET_REFS}" (at 189.2271 34.29 0)
+      (effects (font (size 1.27 1.27)) (justify right) hide)
     )
   )
@@
     )
   )
-  (global_label "SCL1" (shape input) (at 267.97 34.29 0) (fields_autoplaced)
-    (effects (font (size 1.27 1.27)) (justify left))
-    (property "Intersheetrefs" "${INTERSHEET_REFS}" (at 275.5929 34.29 0)
-      (effects (font (size 1.27 1.27)) (justify left) hide)
+  (global_label "SCL1" (shape input) (at 242.57 34.29 180) (fields_autoplaced)
+    (effects (font (size 1.27 1.27)) (justify right))
+    (property "Intersheetrefs" "${INTERSHEET_REFS}" (at 234.9471 34.29 0)
+      (effects (font (size 1.27 1.27)) (justify right) hide)
     )
   )
@@
     )
   )
-  (global_label "SDA1" (shape bidirectional) (at 242.57 34.29 180) (fields_autoplaced)
-    (effects (font (size 1.27 1.27)) (justify right))
-    (property "Intersheetrefs" "${INTERSHEET_REFS}" (at 233.7753 34.29 0)
-      (effects (font (size 1.27 1.27)) (justify right) hide)
+  (global_label "SDA1" (shape bidirectional) (at 267.97 34.29 0) (fields_autoplaced)
+    (effects (font (size 1.27 1.27)) (justify left))
+    (property "Intersheetrefs" "${INTERSHEET_REFS}" (at 276.7647 34.29 0)
+      (effects (font (size 1.27 1.27)) (justify left) hide)
     )
   )
@@
     )
   )
-  (global_label "SDA2" (shape bidirectional) (at 196.85 34.29 180) (fields_autoplaced)
-    (effects (font (size 1.27 1.27)) (justify right))
-    (property "Intersheetrefs" "${INTERSHEET_REFS}" (at 188.0553 34.29 0)
-      (effects (font (size 1.27 1.27)) (justify right) hide)
-    )
-  )
+  (global_label "SDA2" (shape bidirectional) (at 222.25 34.29 0) (fields_autoplaced)
+    (effects (font (size 1.27 1.27)) (justify left))
+    (property "Intersheetrefs" "${INTERSHEET_REFS}" (at 231.0447 34.29 0)
+      (effects (font (size 1.27 1.27)) (justify left) hide)
+    )
+  )
